File: PCB/can2usb/_autosave-can2usb.sch (KiCad schematic (older format))
At the start: 40 parts, among them J1 STLINK, J2 Conn_01x03_Male, P1 USB_C_Plug_USB2.0, U1 STM32F103C6Tx, U2 TLP175A, U3 MCP2561-E-SN, U5 USBLC6-2SC6, U6 MIC5528-3.3YMT-TR, Y1 16MHz, Y2 32KHz

Commit message: New PCB design
Parts:
- gave numbers to parts that had none: 1
Changed lines of the file:
@@
 $EndComp
 $Comp
-L Mechanical:MountingHole H?
+L Mechanical:MountingHole H4
 U 1 1 63501990
 P 7525 6250
-F 0 "H?" H 7625 6296 50  0000 L CNN
+F 0 "H4" H 7625 6296 50  0000 L CNN
 F 1 "MountingHole" H 7625 6205 50  0000 L CNN
 F 2 "MountingHole:MountingHole_2.2mm_M2" H 7525 6250 50  0001 C CNN
